File: KiCAD/espTemp/espTemp.sch (KiCad schematic (older format))
At the start: 7 parts, among them U1 ESP-01, U2 LD1117S33TR_SOT223, U3 DHT11

Commit message: kicad
Parts:
- U2: footprint My_Parts:TO-220F-3_Vertical_large -> My_Misc:TO-220F-3_Horizontal_TabDown_large
Changed lines of the file:
@@
 F 0 "U2" H 6050 2142 50  0000 C CNN
 F 1 "LD1117S33TR_SOT223" H 6050 2051 50  0000 C CNN
-F 2 "My_Parts:TO-220F-3_Vertical_large" H 6050 2100 50  0001 C CNN
+F 2 "My_Misc:TO-220F-3_Horizontal_TabDown_large" H 6050 2100 50  0001 C CNN
 F 3 "http://www.st.com/st-web-ui/static/active/en/resource/technical/document/datasheet/CD00000544.pdf" H 6150 1650 50  0001 C CNN
 	1    6050 1900

Commit message: now dht22
Parts:
- removed U3: DHT11, My_Misc:DHT22,RHT03,CM2303_large, symbol Sensor:DHT11
- added U3: DHT22,CM2303, My_Misc:DHT22,RHT03,CM2303_large, symbol My_Parts:DHT22,CM2303
Changed lines of the file:
@@
-$EndComp
-$Comp
-L Sensor:DHT11 U3
-U 1 1 61A673A0
-P 7950 3150
-F 0 "U3" H 7706 3196 50  0000 R CNN
-F 1 "DHT11" H 7706 3105 50  0000 R CNN
-F 2 "My_Misc:DHT22,RHT03,CM2303_large" H 7950 2750 50  0001 C CNN
-F 3 "http://akizukidenshi.com/download/ds/aosong/DHT11.pdf" H 8100 3400 50  0001 C CNN
-	1    7950 3150
-	1    0    0    -1
 $EndComp
 $Comp
@@
 	8650 3150 8450 3150
 Connection ~ 8450 3150
+$Comp
+L My_Parts:DHT22,CM2303 U3
+U 1 1 61B915F0
+P 7950 3150
+F 0 "U3" H 7707 3196 50  0000 R CNN
+F 1 "DHT22,CM2303" H 7707 3105 50  0000 R CNN
+F 2 "My_Misc:DHT22,RHT03,CM2303_large" H 7950 2750 50  0001 C CNN
+F 3 "http://akizukidenshi.com/download/ds/aosong/DHT11.pdf" H 8100 3400 50  0001 C CNN
+	1    7950 3150
+	1    0    0    -1
+$EndComp
 $EndSCHEMATC

Commit message: DHT22, DHT type
Connections:
- net labels added: GPIO2
- net labels removed: GPIO1
Changed lines of the file:
@@
 L power:GND #PWR0105
 U 1 1 61A926AA
-P 4350 4050
-F 0 "#PWR0105" H 4350 3800 50  0001 C CNN
-F 1 "GND" H 4355 3877 50  0000 C CNN
-F 2 "" H 4350 4050 50  0001 C CNN
-F 3 "" H 4350 4050 50  0001 C CNN
-	1    4350 4050
+P 3950 4050
+F 0 "#PWR0105" H 3950 3800 50  0001 C CNN
+F 1 "GND" H 3955 3877 50  0000 C CNN
+F 2 "" H 3950 4050 50  0001 C CNN
+F 3 "" H 3950 4050 50  0001 C CNN
+	1    3950 4050
 	1    0    0    -1
 $EndComp
@@
 $EndComp
 Wire Wire Line
-	4650 3550 4350 3550
-Wire Wire Line
-	4350 3550 4350 4050
+	3950 3550 3950 4050
 Wire Wire Line
 	6200 3850 6850 3850
@@
 	6850 3650 6850 3850
 Text GLabel 8650 3150 2    50   Input ~ 0
-GPIO1
-Text GLabel 6400 3550 2    50   Input ~ 0
-GPIO1
-Wire Wire Line
-	6200 3550 6400 3550
+GPIO2
+Text GLabel 4450 3650 0    50   Input ~ 0
+GPIO2
 Wire Wire Line
 	8650 3150 8450 3150
@@
 	1    0    0    -1
 $EndComp
+Wire Wire Line
+	3950 3550 4650 3550
+Wire Wire Line
+	4650 3650 4450 3650
 $EndSCHEMATC

Commit message: 100mil DHT on PCB
Parts:
- U3: footprint My_Misc:DHT22,RHT03,CM2303_large -> My_Parts:DHT22,RHT03,CM2303_100mil_large
Changed lines of the file:
@@
 F 0 "U3" H 7707 3196 50  0000 R CNN
 F 1 "DHT22,CM2303" H 7707 3105 50  0000 R CNN
-F 2 "My_Misc:DHT22,RHT03,CM2303_large" H 7950 2750 50  0001 C CNN
+F 2 "My_Parts:DHT22,RHT03,CM2303_100mil_large" H 7950 2750 50  0001 C CNN
 F 3 "http://akizukidenshi.com/download/ds/aosong/DHT11.pdf" H 8100 3400 50  0001 C CNN
 	1    7950 3150
