File: KiCAD/espTemp/espTemp.kicad_sch (KiCad schematic)
At the start: 7 parts, among them U1 ESP-01, U2 LD1117S33TR_SOT223, U3 DHT22,CM2303

Commit message: fixed kicad
Parts:
- removed C2: 10u, My_Misc:CP_Radial_D5.0mm_P2.50mm_larger_pads, symbol Device:CP
- added C2: 10u, My_Misc:CP_Radial_D5.0mm_P2.50mm_larger_pads, symbol Device:C_Polarized
Connections:
- net +3V3: now also C2.1
- net GND: now also C2.2
Changed lines of the file:
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@@
-    (pin "2")
-  )
-  (symbol (lib_id "Device:CP") (at 166.37 57.15 0) (unit 1)
-    (in_bom yes) (on_board yes)
-    (property "Reference" "C2" (id 0) (at 169.3672 55.9816 0)
-      (effects (font (size 1.27 1.27)) (justify left))
-    )
-    (property "Value" "10u" (id 1) (at 169.3672 58.293 0)
-      (effects (font (size 1.27 1.27)) (justify left))
-    )
-    (property "Footprint" "My_Misc:CP_Radial_D5.0mm_P2.50mm_larger_pads" (id 2) (at 167.3352 60.96 0)
-      (effects (font (size 1.27 1.27)) hide)
-    )
-    (property "Datasheet" "~" (id 3) (at 166.37 57.15 0)
-      (effects (font (size 1.27 1.27)) hide)
-    )
-    (pin "1")
     (pin "2")
   )
@@
     (pin "4")
   )
+  (symbol (lib_id "Device:C_Polarized") (at 166.37 57.15 0) (unit 1)
+    (in_bom yes) (on_board yes) (fields_autoplaced)
+    (property "Reference" "C2" (id 0) (at 169.291 55.3525 0)
+      (effects (font (size 1.27 1.27)) (justify left))
+    )
+    (property "Value" "10u" (id 1) (at 169.291 58.1276 0)
+      (effects (font (size 1.27 1.27)) (justify left))
+    )
+    (property "Footprint" "My_Misc:CP_Radial_D5.0mm_P2.50mm_larger_pads" (id 2) (at 167.3352 60.96 0)
+      (effects (font (size 1.27 1.27)) hide)
+    )
+    (property "Datasheet" "~" (id 3) (at 166.37 57.15 0)
+      (effects (font (size 1.27 1.27)) hide)
+    )
+    (pin "1")
+    (pin "2")
+  )
   (sheet_instances
     (path "/" (page "1"))
@@
       (reference "C1") (unit 1) (value "100n") (footprint "My_Misc:C_Disc_D3.0mm_W1.6mm_P2.50mm_larg")
     )
-    (path "/00000000-0000-0000-0000-000061a7af7d"
+    (path "/ac780ebe-5afd-4e74-82f8-509da8ddaa4d"
       (reference "C2") (unit 1) (value "10u") (footprint "My_Misc:CP_Radial_D5.0mm_P2.50mm_larger_pads")
     )

Commit message: 3d view
Parts:
- U1: footprint My_Arduino:ESP-01_large -> My_Arduino:ESP-01_w_pin_socket_large
- U2: footprint My_Misc:TO-220F-3_Horizontal_TabDown_large -> My_Misc:TO-220-3_Horizontal_TabDown_large
- U3: footprint My_Parts:DHT22,RHT03,CM2303_large -> My_Parts:DHT22,RHT03,CM2303_100mil_large
Connections:
- net GPIO2 renamed TempSignal
Changed lines of the file:
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@@
     (stroke (width 0) (type default) (color 0 0 0 0))
   )
-  (wire (pts (xy 100.33 90.17) (xy 118.11 90.17))
+  (wire (pts (xy 95.25 90.17) (xy 118.11 90.17))
     (stroke (width 0) (type default) (color 0 0 0 0))
   )
@@
     (stroke (width 0) (type default) (color 0 0 0 0))
   )
-  (wire (pts (xy 100.33 90.17) (xy 100.33 102.87))
+  (wire (pts (xy 95.25 90.17) (xy 95.25 102.87))
     (stroke (width 0) (type default) (color 0 0 0 0))
   )
@@
     (stroke (width 0) (type default) (color 0 0 0 0))
   )
-  (global_label "GPIO2" (shape input) (at 219.71 80.01 0) (fields_autoplaced)
+  (global_label "TempSignal" (shape input) (at 219.71 80.01 0) (fields_autoplaced)
     (effects (font (size 1.27 1.27)) (justify left))
-    (property "Intersheet References" "${INTERSHEET_REFS}" (id 0) (at 0 0 0)
-      (effects (font (size 1.27 1.27)) hide)
-    )
-  )
-  (global_label "GPIO2" (shape input) (at 113.03 92.71 180) (fields_autoplaced)
+    (property "Intersheet References" "${INTERSHEET_REFS}" (id 0) (at 232.8594 79.9306 0)
+      (effects (font (size 1.27 1.27)) (justify left) hide)
+    )
+  )
+  (global_label "TempSignal" (shape input) (at 113.03 92.71 180) (fields_autoplaced)
     (effects (font (size 1.27 1.27)) (justify right))
-    (property "Intersheet References" "${INTERSHEET_REFS}" (id 0) (at 0 0 0)
-      (effects (font (size 1.27 1.27)) hide)
+    (property "Intersheet References" "${INTERSHEET_REFS}" (id 0) (at 99.8806 92.6306 0)
+      (effects (font (size 1.27 1.27)) (justify right) hide)
     )
   )
@@
     (property "Reference" "U1" (id 0) (at 137.795 84.455 0))
     (property "Value" "ESP-01" (id 1) (at 137.795 86.7664 0))
-    (property "Footprint" "My_Arduino:ESP-01_large" (id 2) (at 135.89 93.98 0)
+    (property "Footprint" "My_Arduino:ESP-01_w_pin_socket_large" (id 2) (at 135.89 93.98 0)
       (effects (font (size 1.27 1.27)) hide)
     )
@@
     (property "Reference" "U2" (id 0) (at 153.67 42.1132 0))
     (property "Value" "LD1117S33TR_SOT223" (id 1) (at 153.67 44.4246 0))
-    (property "Footprint" "My_Misc:TO-220F-3_Horizontal_TabDown_large" (id 2) (at 153.67 43.18 0)
+    (property "Footprint" "My_Misc:TO-220-3_Horizontal_TabDown_large" (id 2) (at 153.67 43.18 0)
       (effects (font (size 1.27 1.27)) hide)
     )
@@
     (pin "2")
   )
-  (symbol (lib_id "power:GND") (at 100.33 102.87 0) (unit 1)
-    (in_bom yes) (on_board yes)
-    (property "Reference" "#PWR0105" (id 0) (at 100.33 109.22 0)
-      (effects (font (size 1.27 1.27)) hide)
-    )
-    (property "Value" "GND" (id 1) (at 100.457 107.2642 0))
-    (property "Footprint" "" (id 2) (at 100.33 102.87 0)
-      (effects (font (size 1.27 1.27)) hide)
-    )
-    (property "Datasheet" "" (id 3) (at 100.33 102.87 0)
+  (symbol (lib_id "power:GND") (at 95.25 102.87 0) (unit 1)
+    (in_bom yes) (on_board yes)
+    (property "Reference" "#PWR0105" (id 0) (at 95.25 109.22 0)
+      (effects (font (size 1.27 1.27)) hide)
+    )
+    (property "Value" "GND" (id 1) (at 95.377 107.2642 0))
+    (property "Footprint" "" (id 2) (at 95.25 102.87 0)
+      (effects (font (size 1.27 1.27)) hide)
+    )
+    (property "Datasheet" "" (id 3) (at 95.25 102.87 0)
       (effects (font (size 1.27 1.27)) hide)
     )
@@
       (effects (font (size 1.27 1.27)) (justify right))
     )
-    (property "Footprint" "My_Parts:DHT22,RHT03,CM2303_large" (id 2) (at 201.93 90.17 0)
+    (property "Footprint" "My_Parts:DHT22,RHT03,CM2303_100mil_large" (id 2) (at 201.93 90.17 0)
       (effects (font (size 1.27 1.27)) hide)
     )
@@
     )
     (path "/00000000-0000-0000-0000-000061a66c7b"
-      (reference "U1") (unit 1) (value "ESP-01") (footprint "My_Arduino:ESP-01_large")
+      (reference "U1") (unit 1) (value "ESP-01") (footprint "My_Arduino:ESP-01_w_pin_socket_large")
     )
     (path "/00000000-0000-0000-0000-000061a79a2b"
-      (reference "U2") (unit 1) (value "LD1117S33TR_SOT223") (footprint "My_Misc:TO-220F-3_Horizontal_TabDown_large")
+      (reference "U2") (unit 1) (value "LD1117S33TR_SOT223") (footprint "My_Misc:TO-220-3_Horizontal_TabDown_large")
     )
     (path "/00000000-0000-0000-0000-000061b915f0"
-      (reference "U3") (unit 1) (value "DHT22,CM2303") (footprint "My_Parts:DHT22,RHT03,CM2303_large")
-    )
-  )
+      (reference "U3") (unit 1) (value "DHT22,CM2303") (footprint "My_Parts:DHT22,RHT03,CM2303_100mil_large")
+    )
+  )
