File: KiCad/espTemp/espTemp.kicad_pcb (KiCad board)
At the start: 2 copper layers, 36.2 x 23.5 mm, 8 parts, among them U1 ESP-01, U2 LD1117S33TR_SOT223, U3 DHT22,CM2303

Commit message: readme and pcb
Parts:
- moved kibuzzard-62077BA3 15.0 mm to (154.3, 86.1)
Changed lines of the file:
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@@
   )
   (footprint "kibuzzard-62077BA3" (layer "F.Cu")
-    (at 141.605 78.105 90)
+    (at 154.305 86.065 90)
     (descr "Converted using: scripting")
     (tags "svg2mod")

Commit message: new pcb, readme
Other:
- board text added: "${TITLE}-${REVISION} Jon Sagebrand github.com/jonsag/espTemp"
- board text removed: "espTemp Jon Sagebrand github.com/jonsag/espTemp"
Changed lines of the file:
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@@
   )
   (paper "A4")
+  (title_block
+    (title "espTemp")
+    (date "2022-12-15")
+    (rev "0.1")
+  )
   (layers
     (0 "F.Cu" signal)
@@
     (effects (font (size 1.5 1.5) (thickness 0.3)) (justify mirror))
   )
-  (gr_text "espTemp\nJon Sagebrand\ngithub.com/jonsag/espTemp" (at 161.29 86.995 -30) (layer "B.Cu")
+  (gr_text "${TITLE}-${REVISION}\nJon Sagebrand\ngithub.com/jonsag/espTemp" (at 161.29 86.995 -30) (layer "B.Cu")
     (effects (font (size 0.635 0.635) (thickness 0.127)) (justify left mirror))
   )
