File: KiCad/espTemp-ams1117/espTemp-ams1117.kicad_sch (KiCad schematic)
At the start: 7 parts, among them U1 ESP-01, U3 DHT22,CM2303

Commit message: kicad v8
Parts:
- BT1: footprint (none) -> My_Headers:2-pin_power_input_header_larger_pads
- C1: footprint (none) -> My_Misc:C_Disc_D3.0mm_W1.6mm_P2.50mm_larg
- C2: footprint (none) -> My_Misc:CP_Radial_D5.0mm_P2.00mm_larger
- U2: value (none) -> AMS1117-3.3; footprint (none) -> Package_TO_SOT_SMD:SOT-223-3_TabPin2
