File: KiCad/espTemp_Screen/espTemp_Screen.kicad_pcb (KiCad board)
At the start: 2 copper layers, 64.8 x 29.2 mm, 9 parts, among them U1 ESP-01, U2 LD1117S33TR_SOT223, U3 DHT22,CM2303, U4 SSD1306_I2C_display

Commit message: new pcb, readme
Other:
- board text added: "${TITLE}-${REVISION} Jon Sagebrand github.com/jonsag/espTemp"
- board text removed: "espTemp Jon Sagebrand github.com/jonsag/espTemp"
Changed lines of the file:
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@@
   )
   (paper "A4")
+  (title_block
+    (title "espTemp-screen")
+    (date "2022-12-15")
+    (rev "0.1")
+  )
   (layers
     (0 "F.Cu" signal)
@@
   (gr_line (start 170.18 102.235) (end 105.41 102.235) (layer "Edge.Cuts") (width 0.05))
   (gr_line (start 105.41 102.235) (end 105.41 73.025) (layer "Edge.Cuts") (width 0.05))
-  (gr_text "espTemp\nJon Sagebrand\ngithub.com/jonsag/espTemp" (at 125.095 83.82 -30) (layer "B.Cu")
+  (gr_text "${TITLE}-${REVISION}\nJon Sagebrand\ngithub.com/jonsag/espTemp" (at 125.095 83.82 -30) (layer "B.Cu")
     (effects (font (size 0.635 0.635) (thickness 0.127)) (justify left mirror))
   )
