File: KiCad/espTemp_Screen/espTemp_Screen.kicad_sch (KiCad schematic)
At the start: 8 parts, among them U1 ESP-01, U2 LD1117S33TR_SOT223, U3 DHT22,CM2303

Commit message: kicad v8
Parts:
- U4: value (none) -> SSD1306_I2C_display; footprint (none) -> My_Parts:SSD1306_I2C_0.96_OLED_display_large
